File: revisions/Backplane_Reference_R2_0/revisions/R2_0/Backplane_Reference_R2_0.brd (EAGLE design)
At the start: 165.1 x 44.5 mm, 52 parts, among them J1 ER2-SHROUD, J10 ER2-SHROUD, J11 ER2-SHROUD, J12 ER2-SHROUD, J13 ER2-SHROUD, J14 ER2-SHROUD, J2 ER2-SHROUD, J3 ER2-SHROUD, J4 ER2-SHROUD, J5 ER2-SHROUD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

Commit message: Update Backplane Reference
Parts:
- removed U$19, U$47: (no value), haycyonmod_Logos:HALCYON_DIAGON
Other:
- board text added: "ERA 2.0 Backplane Reference Design"
- board text removed: "ER 2.0 Backplane Reference Design"
- board text removed: "Halcyon Modular, LLC"
Changed lines of the file:
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@@
 <text x="129.159" y="1.651" size="1.27" layer="21" font="vector" ratio="20" rot="R180">-12V</text>
 <text x="117.983" y="44.196" size="1.27" layer="21" font="vector" ratio="20" rot="R180">GTO</text>
-<text x="132.207" y="0.635" size="1.016" layer="21" font="vector" ratio="20">ER 2.0
+<text x="132.207" y="0.635" size="1.016" layer="21" font="vector" ratio="20">ERA 2.0
 Backplane
 Reference
 Design</text>
-<text x="142.494" y="0.635" size="1.016" layer="22" font="vector" ratio="20" rot="MR0">ER 2.0
+<text x="142.494" y="0.635" size="1.016" layer="22" font="vector" ratio="20" rot="MR0">ERA 2.0
 Backplane
 Reference
 Design</text>
-<text x="61.595" y="5.207" size="1.016" layer="22" font="vector" ratio="20" rot="MR180">Halcyon
-Modular,
-   LLC</text>
-<text x="70.612" y="5.207" size="1.016" layer="21" font="vector" ratio="20" rot="R180">Halcyon
-Modular,
-   LLC</text>
 <text x="51.435" y="-8.001" size="1.778" layer="51" font="vector" ratio="20">Tom Moxon</text>
 </plain>
@@
 <attribute name="VALUE" x="124.333" y="42.164" size="0.889" layer="27" font="vector" ratio="20"/>
 </element>
-<element name="U$19" library="haycyonmod_Logos" package="HALCYON_DIAGON" value="" x="75.438" y="14.859"/>
-<element name="U$47" library="haycyonmod_Logos" package="HALCYON_DIAGON" value="" x="90.678" y="14.986" rot="MR0"/>
 <element name="U$48" library="PatternAgents-Logos" package="BY_CC_SA_TEXT" value="BY_CC_SA_TEXTTEXT" x="20.828" y="-7.874"/>
 <element name="J1" library="ER2" package="ER2" value="ER2-SHROUD" x="8.001" y="22.225" smashed="yes" rot="R90">
