File: revisions/Module_Templates_1U/examples/BAM/BAM_SIMPLE_1U_6HP.brd (EAGLE design)
At the start: 29.5 x 28.4 mm, 6 parts, among them J2 ER2-SHROUD

Commit message: Update Backplane Reference
Other:
- board text removed: "Halcyon Modular"
Changed lines of the file:
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@@
 <setting verticaltext="up"/>
 </settings>
-<grid distance="10" unitdist="mil" unit="mil" style="lines" multiple="10" display="yes" altdistance="0.025" altunitdist="inch" altunit="inch"/>
+<grid distance="10" unitdist="mil" unit="mm" style="lines" multiple="10" display="yes" altdistance="0.025" altunitdist="inch" altunit="inch"/>
 <layers>
 <layer number="1" name="Top" color="4" fill="1" visible="yes" active="yes"/>
@@
 <layer number="220" name="220bmp" color="21" fill="1" visible="no" active="no"/>
 <layer number="221" name="221bmp" color="22" fill="1" visible="no" active="no"/>
-<layer number="222" name="222bmp" color="23" fill="1" visible="no" active="no"/>
 <layer number="223" name="223bmp" color="24" fill="1" visible="no" active="no"/>
 <layer number="224" name="224bmp" color="25" fill="1" visible="no" active="no"/>
@@
 <text x="5.334" y="25.908" size="0.8128" layer="22" font="vector" ratio="20" rot="MR0">RED
 STRIPE</text>
-<text x="23.622" y="25.146" size="1.27" layer="21" font="vector" ratio="20" rot="R180">Halcyon Modular</text>
 <text x="25.4" y="8.89" size="1.27" layer="22" font="vector" ratio="20" rot="R180">Bus Access Module</text>
-<text x="6.604" y="34.29" size="1.27" layer="22" font="vector" ratio="20" rot="SR0">Halcyon Modular</text>
 <text x="23.114" y="19.05" size="1.016" layer="21" font="vector" ratio="20" rot="R180">Bus Access Module</text>
 <text x="1.27" y="19.812" size="1.27" layer="21" font="vector" ratio="20">ERA
