File: revisions/Module_Templates_1U/examples/BAM/BAM_SIMPLE_1U_6HP.sch (EAGLE design)
At the start: 6 parts, among them J2 ER2-SHROUD

Commit message: Update Backplane Reference
Other:
- note added: "Tom Moxon, Patternagents, LLC"
- note removed: "Tom Moxon, Halcyon Modular, LLC"
Changed lines of the file:
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@@
 in 1U and 6 HP size format.
 A single, simple, passive PCB. </text>
-<text x="27.94" y="5.08" size="2.54" layer="91" font="vector" ratio="20">Tom Moxon, Halcyon Modular, LLC</text>
+<text x="27.94" y="5.08" size="2.54" layer="91" font="vector" ratio="20">Tom Moxon, Patternagents, LLC</text>
 </plain>
 <instances>
