File: revisions/Module_Templates_1U/examples/BUF/BUF_1U_6HP_fpb.sch (EAGLE design)
At the start: 11 parts, among them J2 ERA-NOSILK

Commit message: Update Backplane Reference
Other:
- note added: "Tom Moxon, PatternAgents, LLC"
- note removed: "Tom Moxon, Halcyon Modular, LLC"
Changed lines of the file:
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@@
 in 1U and 6 HP size format.
 A single, simple, passive PCB. </text>
-<text x="27.94" y="5.08" size="2.54" layer="91" font="vector" ratio="20">Tom Moxon, Halcyon Modular, LLC</text>
+<text x="27.94" y="5.08" size="2.54" layer="91" font="vector" ratio="20">Tom Moxon, PatternAgents, LLC</text>
 </plain>
 <instances>
