File: revisions/Module_Templates_1U/examples/BUF/BUF_1U_6HP_panel.sch (EAGLE design)
At the start: 1 part

Commit message: Update Backplane Reference
Other:
- note removed: ""4 Jacks - Halcyon Spacing!!!""
Changed lines of the file:
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@@
 <text x="30.48" y="7.62" size="1.9304" layer="91" font="vector" ratio="20">Tom Moxon</text>
 <text x="177.8" y="27.94" size="3.81" layer="91" font="vector" ratio="20">ERA 1U 6HP 4J</text>
-<text x="157.48" y="38.1" size="3.81" layer="91" font="vector" ratio="20">"4 Jacks - Halcyon Spacing!!!"</text>
 </plain>
 <instances>
