File: revisions/Module_Templates_3U/examples/SwitchMult/SwitchMult.brd (EAGLE design)
At the start: 100 x 19.6 mm, 18 parts, among them J1 ERA-SHROUD, P1 PJ301_THONKICONN6, P2 PJ301_THONKICONN6, P3 PJ301_THONKICONN6, P4 PJ301_THONKICONN6, P5 PJ301_THONKICONN6, P6 PJ301_THONKICONN6, P7 PJ301_THONKICONN6, SW1 LP4EE1PBCTG, SW2 LP4EE1PBCTG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

Commit message: Update Backplane Reference
Parts:
- removed R5: 560, halcyonmod_Passives:AXIAL-0.4
- removed SW5: LP4EE1PBCTG, og-switch:LP4OA1PBCT
- added P8: PJ301_THONKICONN6, og-pj301:WQP_PJ_301M6
- moved P6 14.0 mm to (37.0, 4.80)
- moved P7 14.0 mm to (23.0, 4.80)
Connections:
- removed net IN5: P5.P3, SW5.P6
- removed net N$10: R5.P$1, SW5.L1
- removed net N$9: SW5.L2, SW5.P2
- net 12V0: no longer R5.P$2
- net GND: now also P8.P1; no longer SW5.P3
- net MIXBUS: now also P5.P2, P8.P3; no longer SW5.P5
Routing:
- net MIXBUS: track 110.9 -> 126.7 mm
- net IN5: track 13.7 -> 0.00 mm
- net N$9: track 7.06 -> 0.00 mm
- net N$10: track 5.03 -> 0.00 mm
- net GND: track 277.3 -> 279.7 mm
- net 12V0: track 95.0 -> 93.7 mm
Other:
- board text added: "Rev 2.0"
- board text removed: "HALCYON MODULAR"
- board text removed: "Rev 1.1"
