File: revisions/Backplane_Reference_R2_0/revisions/R2_1/Backplane_Compact_R2_1.brd (EAGLE design)
At the start: 96.5 x 85.5 mm, 56 parts, among them J1 ERA-SHROUD, J10 ERA-SHROUD, J11 ERA-SHROUD, J12 ERA-SHROUD, J13 ERA-SHROUD, J14 ERA-SHROUD, J15 ERA-SHROUD, J16 ERA-SHROUD, J2 ERA-SHROUD, J3 ERA-SHROUD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

Commit message: Update Backplane Reference
Parts:
- removed U$10: (no value), haycyonmod_Logos:HALCYON1
- removed U$47: (no value), haycyonmod_Logos:HALCYON_DIAGON
- added U$37: PA_LOGO_SYMMED, PatternAgents-Logos:PA_LOGO_AGENT_MED_SYM
- added U$38: PA_LOGO_SYMLARGE, PatternAgents-Logos:PA_LOGO_AGENT_LRG_SYM
- U$19: value (none) -> PA_LOGO_SYMMED; device haycyonmod_Logos:HALCYON_DIAGON -> PatternAgents-Logos:PA_LOGO_AGENT_MED_SYM
- moved U$19 34.8 mm to (48.5, 69.2), flipped to the bottom
Other:
- board text removed: "Halcyon Modular, LLC"
