File: revisions/Backplane_Reference_R2_0/Backplane.sch (EAGLE design)
At the start: 26 parts, among them Q1 BSS138W-7-F, Q2 BSS138W-7-F

Commit message: 4/10 update
Parts:
- removed CV_IN, GATE_IN: JACK-3_5MM-MONO-SW-MJ_3502, oXo_Connectors:JACK-3_5MM-MONO-SW-MJ_3502
- removed CV_OUT, CV_THRU, GATE_OUT, GATE_THRU: JACK-3_5MM-MONO-SW-MJ_3502, halcyonmod_Connectors:JACK-3_5MM-MONO-SW-MJ_3502
- removed ERA, EURO: ERA-SHROUD, ERA:ERA-SHROUD
- removed FID1, FID2, FID3, FID4: FIDUCIALUFIDUCIAL, TSOC-ESP8266-BASE:FIDUCIALUFIDUCIAL
- removed LED1: LED-RG-CC-PTH-G18500, halcyonmod_Optoelectronics:LED-RG-CC-PTH-G18500
- removed Q1, Q2: BSS138W-7-F, Seeed-Transistor-2016:SMD-MOSFET-N-CH-50V-200MA-BSS138W-7-F(SOT-23)
- removed R4: 1K, halcyonmod_Passives:RESISTOR0603
- removed R5: 4K7, halcyonmod_Passives:RESISTOR0603
- removed R6: 100K, halcyonmod_Passives:RESISTOR0603
- removed U$1, U$2: PA_LOGO_SYMMED, PatternAgents-Logos:PA_LOGO_SYMMED
- added C1, C12, C4, C5, C8, C9: 100nF, PatternAgents-ProtoPads:CAP0603-CAP
- added C10, C11, C2, C3, C6, C7: 100uf, Seeed-Capacitor-2016:DIP-ALUMINUM-100UF-16V(D5-H7MM)
- added D1: Yellow, SparkFun-LED:LED-YELLOW0603
- added D2: RED, SparkFun-LED:LED-RED0603
- added D3: GREEN, SparkFun-LED:LED-GREEN0603
- added H10, H3, H4, H5, H6, H7, H8, H9: MOUNT-HOLE2.8, euro_rack:MOUNT-HOLE2.8
- added J1, J10, J11, J12, J13, J14, J15, J16, J2, J3, J4, J5, J6, J7, J8, J9: ERA-SHROUD, ERA:ERA-SHROUD
- added P1, P2, P3, P4: GREEN-2P-5.0, Seeed-Connector -2016:SCREW-TERMINAL-GREEN(2P-5.0)
- added U$19, U$37: PA_LOGO_SYMMED, PatternAgents-Logos:PA_LOGO_SYMMED
- added U$38: PA_LOGO_SYMLARGE, PatternAgents-Logos:PA_LOGO_SYMLARGE
- H1, H2: value MOUNT-HOLE3,2S -> MOUNT-HOLE2.8; device oXo_Hardware:MOUNT-HOLE3,2S -> euro_rack:MOUNT-HOLE2.8
- R1: value 100K -> 2.2K
- R2: value 1K -> 680R
- R3: value 4K7 -> 2.2K
Connections:
- removed net 12V0_ERA: ERA.10, ERA.9, EURO.10, EURO.9
- removed net 5V0_ERA: ERA.11, ERA.12, EURO.11, EURO.12, Q1.D, Q2.D
- removed net CVI_ERA: CV_IN.TIP, CV_THRU.TIP, ERA.14, R5.2
- removed net CVO_ERA: CV_OUT.TIP, ERA.13
- removed net CVO_ERA_NORM: CV_OUT.TIP_SW
- removed net GTI_ERA: ERA.16, GATE_IN.TIP, GATE_THRU.TIP, R3.2
- removed net GTO_ERA: ERA.15, GATE_OUT.TIP
- removed net GTO_ERA_NORM: GATE_OUT.TIP_SW
- removed net N$1: LED1.GREEN_CATHODE, R2.1
- removed net N$2: LED1.RED_CATHODE, R4.1
- removed net N$3: Q1.G, R3.1
- removed net N$4: Q2.S, R4.2
- removed net N$5: Q2.G, R5.1
- removed net N$6: Q1.S, R2.2
- removed net N$7: CV_IN.TIP_SW, R6.2
- removed net N$8: GATE_IN.TIP_SW, R1.2
- removed net N12V0_ER2: ERA.1, ERA.2, EURO.1, EURO.2
- removed net SCL_ERA: ERA.8
- removed net SDA_ERA: ERA.7
- new net 12V0: C1.1, C10.+, C2.+, C9.1, J1.10, J1.9, J10.10, J10.9, J11.10, J11.9, J12.10, J12.9, J13.10, J13.9, J14.10, J14.9, J15.10, J15.9, J16.10, J16.9, J2.10, J2.9, J3.10, J3.9, J4.10, J4.9, J5.10, J5.9, J6.10, J6.9, J7.10, J7.9, J8.10, J8.9, J9.10, J9.9, P1.1, P2.1, R1.2
- new net 5V0: C5.1, C6.+, C7.+, C8.1, J1.11, J1.12, J10.11, J10.12, J11.11, J11.12, J12.11, J12.12, J13.11, J13.12, J14.11, J14.12, J15.11, J15.12, J16.11, J16.12, J2.11, J2.12, J3.11, J3.12, J4.11, J4.12, J5.11, J5.12, J6.11, J6.12, J7.11, J7.12, J8.11, J8.12, J9.11, J9.12, P1.2, P2.2, R2.2
- new net CVI: J1.14, J2.14, J3.14, J4.14, J5.14, J6.14, J7.14, J8.14
- new net CVI1: J10.14, J11.14, J12.14, J13.14, J14.14, J15.14, J16.14, J9.14
- new net CVO: J1.13, J2.13, J3.13, J4.13, J5.13, J6.13, J7.13, J8.13
- new net CVO1: J10.13, J11.13, J12.13, J13.13, J14.13, J15.13, J16.13, J9.13
- new net GREEN: D3.C, R3.1
- new net GTI: J1.16, J2.16, J3.16, J4.16, J5.16, J6.16, J7.16, J8.16
- new net GTI1: J10.16, J11.16, J12.16, J13.16, J14.16, J15.16, J16.16, J9.16
- new net GTO: J1.15, J2.15, J3.15, J4.15, J5.15, J6.15, J7.15, J8.15
- new net GTO1: J10.15, J11.15, J12.15, J13.15, J14.15, J15.15, J16.15, J9.15
- new net N12V0: C11.-, C12.1, C3.-, C4.1, J1.1, J1.2, J10.1, J10.2, J11.1, J11.2, J12.1, J12.2, J13.1, J13.2, J14.1, J14.2, J15.1, J15.2, J16.1, J16.2, J2.1, J2.2, J3.1, J3.2, J4.1, J4.2, J5.1, J5.2, J6.1, J6.2, J7.1, J7.2, J8.1, J8.2, J9.1, J9.2, P3.2, P4.2, R3.2
- new net RED: D2.A, R2.1
- new net SCL: J1.8, J2.8, J3.8, J4.8, J5.8, J6.8, J7.8, J8.8
- new net SCL1: J10.8, J11.8, J12.8, J13.8, J14.8, J15.8, J16.8, J9.8
- new net SDA: J1.7, J2.7, J3.7, J4.7, J5.7, J6.7, J7.7, J8.7
- new net SDA1: J10.7, J11.7, J12.7, J13.7, J14.7, J15.7, J16.7, J9.7
- new net YELLOW: D1.A, R1.1
- net GND: now also C1.2, C10.-, C11.+, C12.2, C2.-, C3.+, C4.2, C5.2, C6.-, C7.-, C8.2, C9.2, D1.C, D2.C, D3.A, J1.3, J1.4, J1.5, J1.6, J10.3, J10.4, J10.5, J10.6, J11.3, J11.4, J11.5, J11.6, J12.3, J12.4, J12.5, J12.6, J13.3, J13.4, J13.5, J13.6, J14.3, J14.4, J14.5, J14.6, J15.3, J15.4, J15.5, J15.6, J16.3, J16.4, J16.5, J16.6, J2.3, J2.4, J2.5, J2.6, J3.3, J3.4, J3.5, J3.6, J4.3, J4.4, J4.5, J4.6, J5.3, J5.4, J5.5, J5.6, J6.3, J6.4, J6.5, J6.6, J7.3, J7.4, J7.5, J7.6, J8.3, J8.4, J8.5, J8.6, J9.3, J9.4, J9.5, J9.6, P3.1, P4.1; no longer CV_IN.SLEEVE, CV_OUT.SLEEVE, CV_THRU.SLEEVE, ERA.3, ERA.4, ERA.5, ERA.6, EURO.3, EURO.4, EURO.5, EURO.6, GATE_IN.SLEEVE, GATE_OUT.SLEEVE, GATE_THRU.SLEEVE, LED1.CATHODE, R1.1, R6.1
Other:
- note added: "Embedded Rack Architecture 2.0 Backplane Reference Design"
- note removed: "Embedded Rack Interface"
- note removed: "Eurorack Power"
- moved on the sheet: H1, H2, R1, R2, R3
