File: revisions/Module_Templates_3U/examples/BAM/BAM_Reference_R2_1.brd (EAGLE design)
At the start: 109.2 x 27.8 mm, 23 parts, among them Q1 BSS138W-7-F, Q2 BSS138W-7-F

Commit message: 4/10 update
Parts:
- added U$1, U$2: PA_LOGO_SYMMED, PatternAgents-Logos:PA_LOGO_AGENT_MED_SYM
- added U$48: BY_CC_SA_TEXTTEXT, PatternAgents-Logos:BY_CC_SA_TEXT
Routing:
- net 5V0_ERA: track 89.9 -> 77.8 mm
- net GND: track 305.1 -> 305.6 mm
Other:
- board text removed: "Halcyon Modular, LLC"
Changed lines of the file:
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@@
 Access
 Module</text>
-<text x="60.452" y="23.368" size="1.27" layer="22" font="vector" ratio="19" rot="MR0">Halcyon
-Modular, LLC</text>
 <text x="58.42" y="2.286" size="1.27" layer="22" font="vector" ratio="19" rot="MR0">Revision 2.1</text>
 <text x="7.874" y="14.732" size="1.6764" layer="22" font="vector" ratio="19" rot="MR90">GATE OUT</text>
@@
 </element>
 <element name="R3" library="halcyonmod_Passives" package="0603-RES" value="4K7" x="55.118" y="16.002" rot="R90"/>
+<element name="U$48" library="PatternAgents-Logos" package="BY_CC_SA_TEXT" value="BY_CC_SA_TEXTTEXT" x="20.828" y="-17.526"/>
+<element name="U$1" library="PatternAgents-Logos" package="PA_LOGO_AGENT_MED_SYM" value="PA_LOGO_SYMMED" x="43.18" y="5.842"/>
+<element name="U$2" library="PatternAgents-Logos" package="PA_LOGO_AGENT_MED_SYM" value="PA_LOGO_SYMMED" x="64.516" y="5.334" rot="MR0"/>
 </elements>
 <signals>
@@
 <wire x1="82.296" y1="3.81" x2="82.296" y2="0.762" width="0.6096" layer="16"/>
 <wire x1="82.296" y1="6.35" x2="82.296" y2="3.81" width="0.6096" layer="16"/>
+<wire x1="52.324" y1="22.098" x2="52.40969375" y2="22.18369375" width="0.1778" layer="1"/>
+<wire x1="54.864" y1="20.574" x2="54.61" y2="20.376" width="0.1778" layer="1"/>
+<wire x1="54.864" y1="20.574" x2="54.864" y2="20.449" width="0.1778" layer="1"/>
 </signal>
 <signal name="CVO_ERA">
@@
 <wire x1="89.916" y1="8.89" x2="89.662" y2="9.144" width="0.6096" layer="16"/>
 <wire x1="89.662" y1="9.144" x2="58.674" y2="9.398" width="0.6096" layer="16"/>
-<via x="26.67" y="9.144" extent="1-16" drill="0.3556"/>
-<wire x1="58.674" y1="9.398" x2="54.104303125" y2="9.36173125" width="0.6096" layer="16"/>
-<wire x1="54.104303125" y1="9.36173125" x2="52.578384375" y2="9.349621875" width="0.6096" layer="16"/>
-<wire x1="52.578384375" y1="9.349621875" x2="26.67" y2="9.144" width="0.6096" layer="16"/>
-<wire x1="26.67" y1="9.144" x2="26.67" y2="6.35" width="0.6096" layer="1"/>
+<via x="26.67" y="9.398" extent="1-16" drill="0.3556"/>
+<wire x1="52.578384375" y1="9.349621875" x2="26.67" y2="9.398" width="0.6096" layer="16"/>
+<wire x1="26.67" y1="9.398" x2="26.67" y2="6.35" width="0.6096" layer="1"/>
 <wire x1="26.67" y1="6.35" x2="26.67" y2="3.81" width="0.6096" layer="1"/>
 <via x="58.674" y="9.398" extent="1-16" drill="0.3556"/>
-<wire x1="58.674" y1="9.398" x2="47.752" y2="9.144" width="0.4064" layer="16"/>
 <contactref element="Q2" pad="3"/>
 <contactref element="Q1" pad="3"/>
@@
 <wire x1="52.324" y1="9.60400625" x2="52.578384375" y2="9.349621875" width="0.4064" layer="1"/>
 <via x="52.578384375" y="9.349621875" extent="1-16" drill="0.3556"/>
-<wire x1="52.578384375" y1="9.349621875" x2="54.09219375" y2="9.349621875" width="0.4064" layer="16"/>
-<wire x1="54.09219375" y1="9.349621875" x2="54.104303125" y2="9.36173125" width="0.4064" layer="16"/>
 <wire x1="89.916" y1="6.35" x2="89.916" y2="3.81" width="0.1778" layer="16"/>
+<wire x1="52.578384375" y1="9.349621875" x2="58.674" y2="9.349621875" width="0.6096" layer="16"/>
+<wire x1="58.674" y1="9.349621875" x2="58.674" y2="9.398" width="0.6096" layer="16"/>
 </signal>
 <signal name="SCL_ERA">
