File: revisions/Module_Templates_3U/examples/midi_block/panel/midi_block_panel.sch (EAGLE design)
At the start: 0 parts

Commit message: 4/10 update
Other:
- note removed: "Olivier Gillet"
- note removed: "Power entry"
- note removed: "cc-by-sa"
- note removed: "ol.gillet@gmail.com"
Changed lines of the file:
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@@
 <sheet>
 <plain>
-<text x="162.56" y="20.32" size="2.54" layer="94">cc-by-sa</text>
-<text x="162.56" y="15.24" size="2.54" layer="94">Olivier Gillet</text>
-<text x="162.56" y="10.16" size="2.54" layer="94">ol.gillet@gmail.com</text>
-<text x="218.44" y="20.32" size="2.54" layer="94">Power entry</text>
 </plain>
 <instances>
