File: revisions/Module_Templates_3U/examples/midi_block/pcb/midi_block.brd (EAGLE design)
At the start: 99.8 x 44.5 mm, 31 parts, among them U1 74HC7014D

Commit message: 4/10 update
Parts:
- added U$6: PA_LOGO_SYMMED, PatternAgents-Logos:PA_LOGO_AGENT_MED_SYM
- U$5: value (none) -> PA_LOGO_SYMMED; device haycyonmod_Logos:HALCYON_LOGO -> PatternAgents-Logos:PA_LOGO_AGENT_MED_SYM
- moved U$5 22.1 mm to (57.9, 16.5)
Changed lines of the file:
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@@
 <grid distance="10" unitdist="mil" unit="mm" style="lines" multiple="10" display="yes" altdistance="0.5" altunitdist="mm" altunit="mm"/>
 <layers>
-<layer number="1" name="Top" color="4" fill="1" visible="no" active="yes"/>
+<layer number="1" name="Top" color="4" fill="1" visible="yes" active="yes"/>
 <layer number="2" name="Route2" color="1" fill="3" visible="no" active="no"/>
 <layer number="3" name="Route3" color="4" fill="3" visible="no" active="no"/>
@@
 <layer number="14" name="Route14" color="1" fill="6" visible="no" active="no"/>
 <layer number="15" name="Route15" color="4" fill="6" visible="no" active="no"/>
-<layer number="16" name="Bottom" color="1" fill="1" visible="no" active="yes"/>
+<layer number="16" name="Bottom" color="1" fill="1" visible="yes" active="yes"/>
 <layer number="17" name="Pads" color="2" fill="1" visible="yes" active="yes"/>
 <layer number="18" name="Vias" color="2" fill="1" visible="yes" active="yes"/>
@@
 <layer number="20" name="Dimension" color="15" fill="1" visible="yes" active="yes"/>
 <layer number="21" name="tPlace" color="7" fill="1" visible="yes" active="yes"/>
-<layer number="22" name="bPlace" color="7" fill="1" visible="no" active="yes"/>
+<layer number="22" name="bPlace" color="7" fill="1" visible="yes" active="yes"/>
 <layer number="23" name="tOrigins" color="15" fill="1" visible="yes" active="yes"/>
-<layer number="24" name="bOrigins" color="15" fill="1" visible="no" active="yes"/>
+<layer number="24" name="bOrigins" color="15" fill="1" visible="yes" active="yes"/>
 <layer number="25" name="tNames" color="7" fill="1" visible="yes" active="yes"/>
-<layer number="26" name="bNames" color="7" fill="1" visible="no" active="yes"/>
+<layer number="26" name="bNames" color="7" fill="1" visible="yes" active="yes"/>
 <layer number="27" name="tValues" color="7" fill="1" visible="yes" active="yes"/>
 <layer number="28" name="bValues" color="7" fill="1" visible="no" active="yes"/>
@@
 <element name="C3" library="halcyonmod_Passives" package="0603-CAP" value="100nf" x="73.914" y="23.622"/>
 <element name="C1" library="halcyonmod_Passives" package="0603-CAP" value="100nf" x="29.464" y="22.352"/>
-<element name="U$5" library="haycyonmod_Logos" package="HALCYON_LOGO" value="" x="73.914" y="1.27" rot="MR0"/>
 <element name="U$7" library="halcyonmod_Hardware" package="PCB-MB-01-SIDE" value="PCB-MB-SIDE" x="3.302" y="8.128" rot="R90"/>
 <element name="U$8" library="halcyonmod_Hardware" package="PCB-MB-01-SIDE" value="PCB-MB-SIDE" x="96.52" y="8.128" rot="R90"/>
+<element name="U$5" library="PatternAgents-Logos" package="PA_LOGO_AGENT_MED_SYM" value="PA_LOGO_SYMMED" x="57.912" y="16.51" rot="MR0"/>
+<element name="U$6" library="PatternAgents-Logos" package="PA_LOGO_AGENT_MED_SYM" value="PA_LOGO_SYMMED" x="58.166" y="16.51"/>
 </elements>
 <signals>
