File: revisions/Module_Templates_3U/examples/midi_block/pcb/midi_block.sch (EAGLE design)
At the start: 30 parts, among them U1 74HC7014D

Commit message: 4/10 update
Parts:
- added U$5, U$6: PA_LOGO_SYMMED, PatternAgents-Logos:PA_LOGO_SYMMED
Changed lines of the file:
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@@
 <part name="U$7" library="halcyonmod_Hardware" deviceset="PCB-MB" device="-SIDE"/>
 <part name="U$8" library="halcyonmod_Hardware" deviceset="PCB-MB" device="-SIDE"/>
+<part name="U$5" library="PatternAgents-Logos" deviceset="PA_LOGO_SYM" device="MED"/>
+<part name="U$6" library="PatternAgents-Logos" deviceset="PA_LOGO_SYM" device="MED"/>
 </parts>
 <sheets>
@@
 <instance part="U$7" gate="G$1" x="83.82" y="5.08"/>
 <instance part="U$8" gate="G$1" x="101.6" y="5.08"/>
+<instance part="U$5" gate="G$1" x="241.3" y="55.88"/>
+<instance part="U$6" gate="G$1" x="241.3" y="55.88"/>
 </instances>
 <busses>
